Commit message: try changing the fixed frame to map (or something else rather than base link

File: src/testbot_description/urdf/test2.urdf (robot description, URDF)
Before this commit: robot test_robot, 4 links, 3 joints
Links:
- removed link link1
- removed link link2
- removed link link3
- removed link link4
- added link base_footprint; visual box size=0.001 0.001 0.001
- added link base_link; collision box size=${base_len} ${base_width} 0.01; visual box size=${base_len} ${base_width} 0.01
- added link caster_wheel; collision sphere radius=${caster_wheel_radius}; visual sphere radius=${caster_wheel_radius}
Joints:
- removed joint joint1
- removed joint joint2
- removed joint joint3
- added joint base_link_joint: type fixed, parent base_footprint, child base_link, origin xyz=0 0 ${wheel_radius + 0.005} rpy=0 0 0
- added joint caster_wheel_joint: type continuous, parent base_link, child caster_wheel, origin xyz=${caster_wheel_joint_offset} 0 -${caster_wheel_radius+0.005} rpy=0 0 0, axis 0 1 0
