Commit message: added base links

File: src/testbot_description/urdf/robot.urdf (robot description, URDF)
Before this commit: robot visual, 4 links, 3 joints
Links:
- added link right_base_inside, mass 10; collision box size=0.05 0.6 0.2; visual box size=0.05 0.6 0.2
- link base_link: geometry collision cylinder length=0 radius=0; visual cylinder length=0 radius=0
- link left_base_outside: geometry collision box size=0.05 0.6 0.2; visual box size=0.05 0.6 0.2
- link right_base_outside: geometry collision box size=0.05 0.6 0.2; visual box size=0.05 0.6 0.2

Commit message: added inside of base

File: src/testbot_description/urdf/robot.urdf (robot description, URDF)
Before this commit: robot visual, 5 links, 3 joints
Links:
- added link left_base_inside, mass 10; collision box size=0.0254 0.4572 0.2; visual box size=0.0254 0.4572 0.2
- link left_base_outside: geometry collision box size=0.0254 0.4572 0.2; visual box size=0.0254 0.4572 0.2
- link right_base_inside: geometry collision box size=0.0254 0.4572 0.2; visual box size=0.0254 0.4572 0.2
- link right_base_outside: geometry collision box size=0.0254 0.4572 0.2; visual box size=0.0254 0.4572 0.2
Joints:
- added joint base_link_to_left_base_inside: type fixed, parent base_link, child left_base_inside, origin xyz=-0.1524 0 0
- added joint base_link_to_right_base_inside: type fixed, parent base_link, child right_base_inside, origin xyz=0.1524 0 0

Commit message: added one wheel

File: src/testbot_description/urdf/robot.urdf (robot description, URDF)
Before this commit: robot visual, 6 links, 5 joints
Links:
- added link left_front_wheel, mass 10; collision cylinder length=0.0254 radius=0.0508; visual cylinder length=0.0254 radius=0.0508
Joints:
- added joint base_link_to_left_front_wheel: type fixed, parent base_link, child left_front_wheel, origin xyz=0.1651 0.2286 0

Commit message: added rotation link control

File: src/testbot_description/urdf/robot.urdf (robot description, URDF)
Before this commit: robot visual, 7 links, 6 joints
Links:
- added link left_back_wheel, mass 10; collision cylinder length=0.0254 radius=0.0508; visual cylinder length=0.0254 radius=0.1524
- added link right_back_wheel, mass 10; collision cylinder length=0.0254 radius=0.0508; visual cylinder length=0.0254 radius=0.1524
- added link right_front_wheel, mass 10; collision cylinder length=0.0254 radius=0.0508; visual cylinder length=0.0254 radius=0.1524
- link left_front_wheel: geometry collision cylinder length=0.0254 radius=0.0508; visual cylinder length=0.0254 radius=0.1524
Joints:
- added joint base_link_to_left_back_wheel: type fixed, parent base_link, child left_back_wheel, origin xyz=0.1905 -0.2286 0 rpy=1.57075 1.57075 0
- added joint base_link_to_right_back_wheel: type fixed, parent base_link, child right_back_wheel, origin xyz=-0.1905 -0.2286 0 rpy=1.57075 1.57075 0
- added joint base_link_to_right_front_wheel: type continuous, parent base_link, child right_front_wheel, origin xyz=-0.1905 0.2286 0 rpy=1.57075 1.57075 0, axis 0 1 0
- joint base_link_to_left_front_wheel: origin xyz=0.1651 0.2286 0 -> xyz=0.1905 0.2286 0 rpy=1.57075 1.57075 0

File: src/testbot_description/urdf/test.urdf (robot description, URDF)
Before this commit: robot visual, 16 links, 15 joints
Links:
- removed link box
- removed link gripper_pole
- removed link head
- removed link left_back_wheel
- removed link left_base
- removed link left_front_wheel
- removed link left_gripper
- removed link left_leg
- removed link left_tip
- removed link right_back_wheel
- removed link right_base
- removed link right_front_wheel
- removed link right_gripper
- removed link right_leg
- removed link right_tip
- added link right_base_outside, mass 10; collision box size=0.0254 0.4572 0.2; visual box size=0.0254 0.4572 0.2
- link base_link: mass None -> 10; geometry collision cylinder length=0 radius=0; visual cylinder length=0 radius=0
Joints:
- removed joint base_to_left_leg
- removed joint base_to_right_leg
- removed joint gripper_extension
- removed joint head_swivel
- removed joint left_back_wheel_joint
- removed joint left_base_joint
- removed joint left_front_wheel_joint
- removed joint left_gripper_joint
- removed joint left_tip_joint
- removed joint right_back_wheel_joint
- removed joint right_base_joint
- removed joint right_front_wheel_joint
- removed joint right_gripper_joint
- removed joint right_tip_joint
- removed joint tobox
- added joint base_link_to_right_base_outside: type fixed, parent base_link, child right_base_outside, origin xyz=0.2286 0 0

Commit message: fixing bugs

File: src/testbot_description/urdf/robot.urdf (robot description, URDF)
Before this commit: robot visual, 10 links, 9 joints
Links:
- link base_link: mass 10 -> None; geometry visual cylinder length=0 radius=0
- link camera_link: mass 10 -> None; geometry visual box size=0.0254 0.1524 0.1143
- link left_back_wheel: mass 10 -> None; geometry visual cylinder length=0.0254 radius=0.1524
- link left_base_inside: mass 10 -> None; geometry visual box size=0.0254 0.4572 0.2
- link left_base_outside: mass 10 -> None; geometry visual box size=0.0254 0.4572 0.2
- link left_front_wheel: mass 10 -> None; geometry visual cylinder length=0.0254 radius=0.1524
- link right_back_wheel: mass 10 -> None; geometry visual cylinder length=0.0254 radius=0.1524
- link right_base_inside: mass 10 -> None; geometry visual box size=0.0254 0.4572 0.2
- link right_base_outside: mass 10 -> None; geometry visual box size=0.0254 0.4572 0.2
- link right_front_wheel: mass 10 -> None; geometry visual cylinder length=0.0254 radius=0.1524
Joints:
- joint base_link_to_left_back_wheel: axis (none) -> 0 1 0; origin xyz=0.1905 -0.2286 0 rpy=1.57075 1.57075 0 -> xyz=0.1905 -0.2286 0.1524 rpy=1.57075 1.57075 0; type fixed -> continuous
- joint base_link_to_left_base_inside: origin xyz=-0.1524 0 0 -> xyz=-0.1524 0 0.1524
- joint base_link_to_left_base_outside: origin xyz=-0.2286 0 0 -> xyz=-0.2286 0 0.1524
- joint base_link_to_left_front_wheel: axis (none) -> 0 1 0; origin xyz=0.1905 0.2286 0 rpy=1.57075 1.57075 0 -> xyz=0.1905 0.2286 0.1524 rpy=1.57075 1.57075 0; type fixed -> continuous
- joint base_link_to_right_back_wheel: axis (none) -> 0 1 0; origin xyz=-0.1905 -0.2286 0 rpy=1.57075 1.57075 0 -> xyz=-0.1905 -0.2286 0.1524 rpy=1.57075 1.57075 0; type fixed -> continuous
- joint base_link_to_right_base_inside: origin xyz=0.1524 0 0 -> xyz=0.1524 0 0.1524
- joint base_link_to_right_base_outside: origin xyz=0.2286 0 0 -> xyz=0.2286 0 0.1524
- joint base_link_to_right_front_wheel: origin xyz=-0.1905 0.2286 0 rpy=1.57075 1.57075 0 -> xyz=-0.1905 0.2286 0.1524 rpy=1.57075 1.57075 0

Commit message: lidar

File: src/testbot_description/urdf/robot.urdf (robot description, URDF)
Before this commit: robot visual, 10 links, 9 joints
Links:
- added link laser
Joints:
- added joint base_link_to_laser: type fixed, parent base_link, child laser, origin xyz=0.0 0.0 0.3 rpy=0.0 0.0 3.14192, axis 0 0 0
