Commit message: working on updated tf

File: src/testbot_description/urdf/nox.urdf (robot description, URDF)
Before this commit: robot nox, 2 links, 1 joints
Joints:
- removed joint base_link_to_zed
- added joint base_link_to_laser: type fixed, parent base_link, child laser, origin xyz=0.0 0.0 0.3 rpy=0.0 0.0 3.14192, axis 0 0 0
